File: basemodule.kicad_sch (KiCad schematic)
At the start: 19 parts, among them J1 Conn_01x05_Pin, J2 USB_C_Receptacle_USB2.0_14P, J3 USB_C_Receptacle_PowerOnly_24P, U1 ESP32-S3-WROOM-1, U2 LD1117S33TR_SOT223, U3 WE-TVS-82400102, U4 CYPD3177-24LQ

Commit message: schematic almost done... the hard part is still in front of us still need to add tantalum or electrolytic caps to output of LD1117
Parts:
- removed J1: Conn_01x05_Pin, symbol Connector:Conn_01x05_Pin
- added C2: 4.7u 25V, symbol Device:C
- added C3, C4: 1u 25V, symbol Device:C
- added C5, C7: 1u, symbol Device:C
- added C6: 22u, symbol Device:C
- added D1: 1N5240B, Diode_THT:D_DO-35_SOD27_P7.62mm_Horizontal, symbol Device:D_Zener
- added D2: LTST-C150CKT, LED_SMD:LED_1206_3216Metric, symbol Device:LED
- added J2: Header_UART, Connector_PinHeader_2.54mm:PinHeader_1x03_P2.54mm_Vertical, symbol Connector_Generic:Conn_01x03
- added J4: Header_SpareGPIO, Connector_PinHeader_2.54mm:PinHeader_1x05_P2.54mm_Vertical, symbol Connector_Generic:Conn_01x05
- added J6: Conn_01x05, symbol Connector_Generic:Conn_01x05
- added Q1, Q2: 2SJ652, symbol Transistor_FET:Q_PMOS_GDS
- added R10, R14, R17: 10k, symbol Device:R
- added R11, R8: 0, symbol Device:R
- added R12: 49.9k, symbol Device:R
- added R13: 300, symbol Device:R
- added R15, R16: 4.7k, symbol Device:R
- added R5, R6: 5.1k, symbol Device:R
- added R7: inf, symbol Device:R
- added R9: 1k, symbol Device:R
- added SW1: SW_Boot, Button_Switch_THT:SW_PUSH_6mm, symbol Switch:SW_Push
- added SW2: SW_Reset, Button_Switch_THT:SW_PUSH_6mm, symbol Switch:SW_Push
- added TP1, TP2, TP3, TP4: TestPoint, symbol Connector:TestPoint
- C1: value 1uf -> 1u
- C10: renamed from C3; value 0.1uf -> 0.1u
- C8: renamed from C1; value 1uf -> 1u
- C9: renamed from C2; value 0.1uf -> 0.1u
- R2: value 5.1k -> 1k
- R3: value 0 -> 5.1k
- R4: value inf -> 1k
- renumbered J2 to J3, J3 to J5, R1 to R18, R2 to R19, U3 to U1, U1 to U2, U2 to U3
Connections:
- net +3V3: now also C6.1, C7.1, J6.3 (Pin_3), R14.1, R15.1, R16.1, R17.2
- net +5V: now also TP1.1
- net 3V3_PDchip: now also R5.1, R7.1
- net GND: now also C5.2, C6.2, C7.2, J2.1 (Pin_1), J4.1 (Pin_1), J6.2 (Pin_2), SW1.2, SW2.2, TP2.1
- net GNDPWR: now also C2.2, R13.2, R6.2, R8.2, TP4.1
- net BOOT: now reaches U2.27 (IO0)
- net BOOT: now also R14.2, SW1.1
- net SPARE_35: now reaches U2.28 (IO35)
- net SPARE_35: now also J4.2 (Pin_2)
- net SPARE_36: now reaches U2.29 (IO36)
- net SPARE_36: now also J4.3 (Pin_3)
- net EN: now reaches U2.3 (EN)
- net EN: now also C5.1, R17.1, SW2.1
- net SPARE_37: now reaches U2.30 (IO37)
- net SPARE_37: now also J4.4 (Pin_4)
- net SPARE_38: now reaches U2.31 (IO38)
- net SPARE_38: now also J4.5 (Pin_5)
- net RXD0: now reaches U2.36 (RXD0)
- net RXD0: now also J2.3 (Pin_3)
- net TXD0: now reaches U2.37 (TXD0)
- net TXD0: now also J2.2 (Pin_2)
- net SDA: now reaches U2.4 (IO4)
- net SDA: now also J6.4 (Pin_4), R15.2
- net SCL: now reaches U2.5 (IO5)
- net SCL: now also J6.5 (Pin_5), R16.2
- net VBUS_CONN: now reaches J5.A4 (VBUS), J5.A9 (VBUS), J5.B4 (VBUS), J5.B9 (VBUS), U4.18 (VBUS_IN)
- net VBUS_CONN: now also C2.1, C3.1, Q1.2 (D), R10.1
- net +9V: now reaches U4.11 (VDC_OUT)
- net +9V: now also C4.1, J6.1 (Pin_1), Q2.2 (D), TP3.1
- net VBUS_FET_EN: now reaches U4.3 (VBUS_FET_EN)
- net VBUS_FET_EN: now also R9.2
- net ISNK_COARSE: now reaches U4.5 (ISNK_COARSE)
- net ISNK_COARSE: now also R5.2, R6.1
- net ISNK_FINE: now reaches U4.6 (ISNK_FINE)
- net ISNK_FINE: now also R7.2, R8.1
- net FAULT: now reaches U4.9 (FAULT)
- net FAULT: now also D2.2 (A)
- new net: D2.1 (K), R13.1
- new net: C3.2, C4.2, R10.2, R11.2, R9.1
- new net FET_GATE: D1.2 (A), Q1.1 (G), Q2.1 (G), R11.1, R12.2
- new net FET_SRC: D1.1 (K), Q1.3 (S), Q2.3 (S), R12.1
- no-connect marks 0 -> 33
Other:
- note added: "Configures for 3A current"
- note added: "Configures for Min and Max voltage of 9V."
- note removed: "This should set Min voltage to 20 and Max voltage to 15. According to datasheet, if min>max, actual min and max voltage are set to the set max voltage."
- company: (none) -> mixer-control
- title: (none) -> Base Module
- moved on the sheet: J5, U2

Commit message: complete
Parts:
- removed U3: LD1117S33TR_SOT223, Package_TO_SOT_SMD:SOT-223-3_TabPin2, symbol Regulator_Linear:LD1117S33TR_SOT223
- added C11: 10u, Capacitor_SMD:C_0805_2012Metric_Pad1.18x1.45mm_HandSolder, symbol Device:C
- added C12: 22u, Capacitor_SMD:C_0805_2012Metric_Pad1.18x1.45mm_HandSolder, symbol Device:C
- added U5: AZ1117-3.3, Package_TO_SOT_SMD:TO-252-2, symbol Regulator_Linear:AZ1117-3.3
- C1, C10, C2, C3, C4, C5, C6, C7, C8, C9: footprint (none) -> Capacitor_SMD:C_0805_2012Metric_Pad1.18x1.45mm_HandSolder
- J3, J5: footprint (none) -> Connector_USB:USB_C_Receptacle_GCT_USB4085
- J6: value Conn_01x05 -> Pogo_Magentic_Out; footprint (none) -> Connector_PinHeader_2.54mm:PinHeader_1x05_P2.54mm_Vertical
- NT1: footprint (none) -> NetTie:NetTie-2_SMD_Pad2.0mm
- Q1, Q2: footprint (none) -> Package_TO_SOT_THT:TO-220F-3_Vertical
- R1, R10, R11, R14, R17, R18, R19, R2, R3, R4, R5, R6, R7, R8, R9: footprint (none) -> Resistor_SMD:R_0805_2012Metric_Pad1.20x1.40mm_HandSolder
- R12: value 49.9k -> 100k; footprint (none) -> Resistor_SMD:R_0805_2012Metric_Pad1.20x1.40mm_HandSolder
- R13: value 300 -> 330; footprint (none) -> Resistor_SMD:R_0805_2012Metric_Pad1.20x1.40mm_HandSolder
- R15, R16: footprint (none) -> Resistor_SMD:R_1206_3216Metric_Pad1.30x1.75mm_HandSolder
- TP1, TP2, TP3, TP4: footprint (none) -> TestPoint:TestPoint_Loop_D2.50mm_Drill1.0mm
Connections:
- net +3V3: now also C12.1, U5.2 (VO)
- net +5V: now also C11.1, U5.3 (VI)
- net GND: now also C11.2, C12.2, U5.1 (GND)
