File: fader_module.kicad_sch (KiCad schematic)
At the start: 8 parts, among them IC1 LMD18245T_NOPB, J4 Conn_01x05_Pin, J5 Conn_01x05_Pin, SW1 1825910-6, U5 ATMEGA328P-AUR

Commit message: wip fader wip
Parts:
- added C10, C11, C12, C13, C4, C7, C8: 0.1uF, symbol Device:C
- added C5: 100uF, symbol Device:C
- added C6, C9: 1uF, symbol Device:C
- added D2: LED, symbol Device:LED
- added R4, R5, R8, R9: 10k, symbol Device:R
- added R6, R7: 330, symbol Device:R
- added SW2: 1825910-6, 1825910-6:SW_1825910-6-4, symbol 1825910-6:1825910-6
Connections:
- net +3V3: now also U5.18 (AVCC), U5.6 (VCC__1), C10.1, C9.1, R8.1, R9.1, SW2.3, SW2.4
- net +9V: now also C11.1, C5.1, C6.1
- net GND: now also IC1.5 (PGND), U5.21 (GND__2), U5.5 (GND__1), C10.2, C11.2, C12.2, C13.2, C4.2, C5.2, C6.2, C7.1, C8.2, C9.2, D2.1 (K), SW2.2
- net LINE: now also R4.1; no longer U5.23 (PC0(ADC0/PCINT8))
- net MUTE: now also C12.1, R8.2
- net SERVO: now also R5.1; no longer U5.24 (PC1(ADC1/PCINT9))
- net TOUCH: now also U5.16 (PB4(PCINT4/MISO)); no longer U5.14 (PB2(PCINT2/~{SS}/OC1B))
- net S_LED: now reaches U5.15 (PB3(PCINT3/OC2A/MOSI))
- net S_LED: now also R7.1
- net at U5.20 (AREF): now also C4.1
- net LED: no longer names the net of D1.2 (A)
- net LED: now also R6.2; no longer U5.13 (PB1(PCINT1/OC1A))
- new net: C8.1, R5.2, U5.24 (PC1(ADC1/PCINT9))
- new net: D2.2 (A), R7.2
- new net: C7.2, R4.2, U5.23 (PC0(ADC0/PCINT8))
- new net M_LED: R6.1, U5.13 (PB1(PCINT1/OC1A))
- new net SOLO: C13.1, R9.2, SW2.1, U5.14 (PB2(PCINT2/~{SS}/OC1B))
Other:
- moved on the sheet: D1, IC1, J4, J5, SW1, U5
